Commit message: Shit is working somehow

File: src/assignment3/Test_Worlds/Models/boundary.urdf (robot description, URDF)
Before this commit: robot boundary, 1 links, 0 joints
Links:
- link box: geometry collision box size=1 1 2; visual box size=1 1 2

File: src/assignment3/Test_Worlds/Models/obstacle.urdf (robot description, URDF)
Before this commit: robot obstacle, 1 links, 0 joints
Links:
- link box: mass 1.0 -> 64.0; geometry collision box size=0.5 0.5 2.0; visual box size=0.5 0.5 2.0

File: src/assignment3/Test_Worlds/Models/rubbish.urdf (robot description, URDF)
Before this commit: robot rubbish, 1 links, 0 joints
Links:
- link box: geometry collision box size=0.25 0.25 2; visual box size=0.25 0.25 2
